File: kicad/ethernet-pmod.kicad_pcb (KiCad board)
At the start: 2 copper layers, 50.8 x 20.3 mm, 26 parts, among them J1 PMOD, J2 RJ45_AMP_RJMG1, J3 MDIO, U1 LAN8720A

Commit message: cleanup: improve PMOD header (J1) presentation in schematic
- tidied up schematic
- added commentary on pin orientation
- renamed RST to RSTn for clarity
- re-exported schematic to PDF
Connections:
- J1 pad 8: /RST -> /RSTn
Routing:
- net /RSTn: track 0.00 -> 25.3 mm, vias 0 -> 1
- net /RST: track 25.3 -> 0.00 mm, vias 1 -> 0
Changed lines of the file:
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@@
   (net 27 "unconnected-(U1-Pad4)")
   (net 28 "Net-(R9-Pad2)")
+  (net 29 "/RSTn")
   (footprint "Capacitor_SMD:C_0402_1005Metric" (layer "F.Cu")
     (at 70.6 60)
@@
       (net 25 "/CLKIN") (pinfunction "Pin_7") (pintype "passive"))
     (pad "8" thru_hole oval locked (at 0 2.54) (size 1.7 1.7) (drill 1) (layers *.Cu *.Mask)
-      (net 6 "/RST") (pinfunction "Pin_8") (pintype "passive"))
+      (net 29 "/RSTn") (pinfunction "Pin_8") (pintype "passive"))
     (pad "9" thru_hole oval locked (at 0 5.08) (size 1.7 1.7) (drill 1) (layers *.Cu *.Mask)
       (net 8 "/TXEN") (pinfunction "Pin_9") (pintype "passive"))
@@
   (segment (start 69.596 64.45048) (end 66.172526 64.45048) (width 0.2) (layer "F.Cu") (net 5))
   (segment (start 56.582 62.23) (end 56.612 62.2) (width 0.2) (layer "F.Cu") (net 5))
-  (segment (start 72.2 66.6) (end 59.037006 66.6) (width 0.2) (layer "F.Cu") (net 6))
-  (segment (start 57.80352 65.366514) (end 57.80352 63.60848) (width 0.2) (layer "F.Cu") (net 6))
-  (segment (start 72.35 65.6375) (end 72.35 66.45) (width 0.2) (layer "F.Cu") (net 6))
-  (segment (start 57.80352 63.60848) (end 57.912 63.5) (width 0.2) (layer "F.Cu") (net 6))
-  (segment (start 72.35 66.45) (end 72.2 66.6) (width 0.2) (layer "F.Cu") (net 6))
-  (segment (start 59.037006 66.6) (end 57.80352 65.366514) (width 0.2) (layer "F.Cu") (net 6))
-  (via (at 57.912 63.5) (size 0.8) (drill 0.4) (layers "F.Cu" "B.Cu") (net 6))
-  (segment (start 53.68925 60.61075) (end 52.7685 59.69) (width 0.2) (layer "B.Cu") (net 6))
-  (segment (start 54.0385 60.96) (end 55.88 60.96) (width 0.2) (layer "B.Cu") (net 6))
-  (segment (start 54.014554 60.936054) (end 53.68925 60.61075) (width 0.2) (layer "B.Cu") (net 6))
-  (segment (start 53.68925 60.61075) (end 54.0385 60.96) (width 0.2) (layer "B.Cu") (net 6))
-  (segment (start 55.88 60.96) (end 57.912 62.992) (width 0.2) (layer "B.Cu") (net 6))
-  (segment (start 57.912 62.992) (end 57.912 63.5) (width 0.2) (layer "B.Cu") (net 6))
   (segment (start 73.35 65.6375) (end 73.35 66.65) (width 0.2) (layer "F.Cu") (net 7))
   (segment (start 58.706994 67.4) (end 56.076994 64.77) (width 0.2) (layer "F.Cu") (net 7))
@@
   (segment (start 65.760674 64.297326) (end 65.262674 64.297326) (width 0.2) (layer "F.Cu") (net 28))
   (segment (start 69.596 63.85) (end 69.438 64.008) (width 0.2) (layer "F.Cu") (net 28))
+  (segment (start 72.2 66.6) (end 59.037006 66.6) (width 0.2) (layer "F.Cu") (net 29))
+  (segment (start 57.80352 65.366514) (end 57.80352 63.60848) (width 0.2) (layer "F.Cu") (net 29))
+  (segment (start 72.35 65.6375) (end 72.35 66.45) (width 0.2) (layer "F.Cu") (net 29))
+  (segment (start 57.80352 63.60848) (end 57.912 63.5) (width 0.2) (layer "F.Cu") (net 29))
+  (segment (start 72.35 66.45) (end 72.2 66.6) (width 0.2) (layer "F.Cu") (net 29))
+  (segment (start 59.037006 66.6) (end 57.80352 65.366514) (width 0.2) (layer "F.Cu") (net 29))
+  (via (at 57.912 63.5) (size 0.8) (drill 0.4) (layers "F.Cu" "B.Cu") (net 29))
+  (segment (start 53.68925 60.61075) (end 52.7685 59.69) (width 0.2) (layer "B.Cu") (net 29))
+  (segment (start 54.0385 60.96) (end 55.88 60.96) (width 0.2) (layer "B.Cu") (net 29))
+  (segment (start 54.014554 60.936054) (end 53.68925 60.61075) (width 0.2) (layer "B.Cu") (net 29))
+  (segment (start 53.68925 60.61075) (end 54.0385 60.96) (width 0.2) (layer "B.Cu") (net 29))
+  (segment (start 55.88 60.96) (end 57.912 62.992) (width 0.2) (layer "B.Cu") (net 29))
+  (segment (start 57.912 62.992) (end 57.912 63.5) (width 0.2) (layer "B.Cu") (net 29))
   (zone (net 1) (net_name "GND") (layer "B.Cu") (hatch edge 0.508)
     (connect_pads (clearance 0.35))
